Commit message: depth camera configured

File: sjtu_drone_description/urdf/sjtu_drone.urdf.xacro (robot description, xacro)
@@ -48,10 +48,10 @@
   </joint>
   <link name="front_cam_link"/>
-    <joint name="front_lidar_joint" type="fixed">
-    <origin rpy="0 0 0" xyz="0.2 0 0"/>
-    <parent link="base_link" />
-    <child link="front_lidar_link" />
-  </joint>
-  <link name="front_lidar_link"/>
+  <joint name="front_cam_optical_joint" type="fixed">
+  <origin rpy="-1.5708 0 -1.5708" xyz="0 0 0"/>
+  <parent link="front_cam_link"/>
+  <child link="front_cam_optical_frame"/>
+  </joint>
+  <link name="front_cam_optical_frame"/>
   <joint name="bottom_cam_joint" type="fixed">
     <origin rpy="0 ${M_PI/2} 0" xyz="0 0 0"/>
@@ -177,18 +177,19 @@
   </gazebo>
   <gazebo reference="front_cam_link">
-  <sensor type="depth" name="front_camera">
-    <update_rate>30.0</update_rate>
-    <visualize>true</visualize>
+    <sensor name="front_camera" type="depth">
+      <always_on>true</always_on>
+      <visualize>true</visualize>
+      <update_rate>30</update_rate>
       <camera>
-        <horizontal_fov>2.09</horizontal_fov>
-        <image>
-          <width>640</width>
-          <height>360</height>
-          <format>R8G8B8</format>
-        </image>
-        <clip>
-          <near>0.1</near>
-          <far>100</far>
-        </clip>
+        <horizontal_fov>1.02974</horizontal_fov>
+          <image>
+            <width>1920</width>
+            <height>1080</height>
+            <format>R8G8B8</format>
+          </image>
+          <clip>
+            <near>0.2</near>
+            <far>300</far>
+          </clip>
         <noise>
           <type>gaussian</type>
@@ -197,20 +198,11 @@
         </noise>
       </camera>
-      <plugin name="depth_camera_controller" filename="libgazebo_ros_camera.so">
-        <ros>
-          <namespace>${mp['namespace']}</namespace>
-        </ros>
-        <frame_name>${mp['namespace']}/front_cam_link</frame_name>
-        <alwaysOn>true</alwaysOn>
-        <updateRate>30.0</updateRate>  <!-- Camera update rate in Hz -->
-        <cameraName>front_depth_camera</cameraName>
-        <imageTopicName>depth/image_raw</imageTopicName>
-        <cameraInfoTopicName>depth/camera_info</cameraInfoTopicName>
-        <hackBaseline>0.07</hackBaseline>  <!-- Adjust baseline for stereo depth cameras -->
-        <horizontal_fov>1.047</horizontal_fov>  <!-- Field of view in radians -->
-        <imageWidth>640</imageWidth>  <!-- Width of the camera image -->
-        <imageHeight>480</imageHeight>  <!-- Height of the camera image -->
-        <nearClip>0.1</nearClip>  <!-- Near clipping distance -->
-        <farClip>100.0</farClip>  <!-- Far clipping distance -->
+      <plugin name="camera_front" filename="libgazebo_ros_camera.so">
+        <ros>
+          <namespace>${mp['namespace']}</namespace>
+        </ros>
+        <frame_name>${mp['namespace']}/front_cam_optical_frame</frame_name>
+        <camera_name>front</camera_name>
+        <hack_baseline>0.07</hack_baseline>
       </plugin>
     </sensor>
@@ -251,5 +243,4 @@
     </sensor>
   </gazebo>
-<!-- Velodyne ending -->
   <gazebo reference="base_link">
     <sensor name="gps" type="gps">
@@ -291,5 +282,4 @@
         <ros>
           <namespace>${mp['namespace']}</namespace>
-          <!-- <remapping>bumper_states:=bumper_states</remapping> -->
         </ros>
         <frame_name>${mp['namespace']}/base_link</frame_name>
